File: HUB75-Sinking_input_screw_terminals/kicad/HUB75-Sinking_input.kicad_pcb (KiCad board)
At the start: 2 copper layers, 85 x 56 mm, 48 parts, among them J1 Conn_01x03_Male, J2 Conn_01x03_Male, J3 Conn_01x03_Male, J4 Conn_01x03_Male, J5 Conn_01x03_Male, J6 TerminalBlock_Phoenix:Termina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, Q1 AO3401A, Q2 2N7002, Q3 2N7002, Q4 2N7002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

Commit message: after the last edits
Other:
- board text added: "HUB-75 SINKING INPUT SCREW TERMINALS V1.0"
- board text removed: "HUB-75 SINKING INPUT V1.0"
Changed lines of the file:
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@@
       (outputformat 1)
       (mirror false)
-      (drillshape 1)
+      (drillshape 0)
       (scaleselection 1)
       (outputdirectory "")
@@
     (effects (font (size 1.524 1.524) (thickness 0.3048)))
   )
-  (gr_text "HUB-75 SINKING INPUT V1.0" (at 87.63 30.48) (layer "F.SilkS")
+  (gr_text "HUB-75 SINKING\nINPUT SCREW\nTERMINALS V1.0" (at 45.72 31.75) (layer "F.SilkS")
     (effects (font (size 1.524 1.524) (thickness 0.3048)))
   )
